File: hardware/kicad/radar_multisim.kicad_sch (KiCad schematic)
At the start: 60 parts, among them T1 lossless, Z0 50, TD 667 ns, T2 lossless, Z0 50, TD 20 ns, U1 TL072CP, U2 TL072CP, X1 0 V -> 1 V in 6.4 ms, repeat, X2 1 -> 5 MHz for 0 -> 1 V, 1 Vpk

Commit message: KiCad: a flow sheet showing how the five test blocks connect
radar_flow.kicad_sch (gen_flow.py) puts blocks 1-5 back together. The
Multisim sheet draws them isolated because that is how you bench them;
this one answers what that sheet cannot: block 5 or the mixer feeds the
IF into block 1, block 3 feeds VANA to blocks 1 and 2, block 2 feeds
VREF to six points inside block 1, and blocks 1 and 4 land on the sound
card's two channels. Every connection carries its level, from +5 dBm out
of the PLL to 19 mV pk at the sound card. Passes the same connectivity
check as the other sheets: no dangling ends, no single-pin nets.

kicad_lib.py: multi-line text broke the KiCad writer, which emitted raw
newlines inside quoted s-expression strings, so any sheet using one
failed to load. Newlines are now escaped, the SVG writer renders them as
tspans instead of collapsing them, and it honours hide_value and the
explicit value/reference positions the writer already accepted.

Beat figures corrected to the 40 MHz coexistence sweep throughout, and
the baseband levels are the ngspice numbers, not estimates.
Parts:
- removed C1 (x2), C2 (x2): 100n, symbol Device:C
- removed C9 (x2): 10n, symbol Device:C
- removed R12 (x2): 1k, symbol Device:R
- removed R2 (x2), R6 (x2), R_LOAD: 10k, symbol Device:R
- removed R_LOAD: 2.2k, symbol Device:R
- removed unit 3 of U2 (x2)
- removed V_ANA (x2): DC 11.4 V, symbol Simulation:VDC
- added C1 (x2), C2 (x2): 100n, symbol Device:C
- added C9 (x2): 10n, symbol Device:C
- added R12 (x2): 1k, symbol Device:R
- added R2 (x2), R6 (x2), R_LOAD: 10k, symbol Device:R
- added R_LOAD: 2.2k, symbol Device:R
- added unit 3 of U2 (x2)
- added V_ANA (x2): DC 11.4 V, symbol Simulation:VDC
Connections:
- net GND: now also C9.2, R2.2, R6.2, R_LOAD.2, R_LOAD.2, U2.4 (V-), U2.4 (V-), V_ANA.2 (-), V_ANA.2 (-)
- net IF_MODEL: now also R12.1
- net TP_AOUT: now also C2.1
- net TP_AP: now also C1.2, R2.1
- net TP_AUDIO: now also R_LOAD.1
- net TP_BEAT: now also C2.2, R6.1
- net TP_BOUT: now also R12.1
- net TP_IF: now also C1.1
- net TP_LP: now also C9.1, R12.2
- net TP_VREF: now also R_LOAD.1
- net VANA: now also U2.8 (V+), U2.8 (V+), V_ANA.1 (+), V_ANA.1 (+)
- net VREF: now also C9.2, R2.2, R6.2
- net at U1.5 (+): now also C2.2, R6.1
- new net: C1.2, C2.1, R2.1
- new net: C1.1, C9.1, R12.2
