File: breadboard/schematics/radar_breadboard.kicad_sch (KiCad schematic)
At the start: 76 parts, among them J1 MIXER IF, J10 ADF LOGIC, J11 A4988 LOGIC, J12 AUDIO R, J2 AUDIO L, J3 12V IN, J4 TO BUCK IN, J5 FROM BUCK 5V, J6 ADF4351 5V, J7 PA 5V, J8 LNA 5V, J9 ESP32, M1 ADF4351 board, M2 3 dB pad, M3 PA module, M4 2-way splitter, M5 band-pass 2400-2500, M6 LNA module, M7 mixer ZX05-43MH-S+, M8 A4988 driver, M9 NEMA-17 stepper, U1 TL072, U2 TL072

Commit message: Add HFSS and Multisim results, report, and the C6 / probe fixes
- report/: short LaTeX write-up of both simulations with all figures
- antenna/: HFSS results (match, gain, patterns, leakage, probe sweep,
  mesh and copper checks), build guide with the new probe position
  (27 mm long, 17.7 mm from the back wall), waterjet cut files
- breadboard/multisim/: the ten Multisim projects, exported data and
  plots, and a results table for every card
- breadboard: C6 raised from 47 uF to 3.3 mF in the layout, wiring
  list, build steps, parts list, schematics and netlists (card 8 showed
  the half-rail reference moving with the signal)
- README: what was simulated, the numbers, and what they mean

Co-Authored-By: Claude Opus 5.5 <noreply@anthropic.com>
Claude-Session: https://claude.ai/code/session_01KoWH1xnrufgnnhp3AGqJnH
Parts:
- C6: value 47u -> 3300u
Changed lines of the file:
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@@
   (symbol (lib_id "Device:C_Polarized") (at 76 122 0) (unit 1) (in_bom yes) (on_board yes) (dnp no)
     (property "Reference" "C6" (at 78.5 120.5 0) (effects (font (size 1.27 1.27)) (justify left)))
-    (property "Value" "47u" (at 78.5 123.5 0) (effects (font (size 1.27 1.27)) (justify left)))
+    (property "Value" "3300u" (at 78.5 123.5 0) (effects (font (size 1.27 1.27)) (justify left)))
     (property "Footprint" "" (at 76 122 0) (effects (font (size 1.27 1.27)) hide))
     (property "Datasheet" "" (at 76 122 0) (effects (font (size 1.27 1.27)) hide))
