File: breadboard/schematics/radar_multisim.kicad_sch (KiCad schematic)
At the start: 60 parts, among them T1 lossless, Z0 50, TD 667 ns, T2 lossless, Z0 50, TD 20 ns, U1 TL072CP, U2 TL072CP, X1 0 V -> 1 V in 6.4 ms, repeat, X2 1 -> 5 MHz for 0 -> 1 V, 1 Vpk

Commit message: Add HFSS and Multisim results, report, and the C6 / probe fixes
- report/: short LaTeX write-up of both simulations with all figures
- antenna/: HFSS results (match, gain, patterns, leakage, probe sweep,
  mesh and copper checks), build guide with the new probe position
  (27 mm long, 17.7 mm from the back wall), waterjet cut files
- breadboard/multisim/: the ten Multisim projects, exported data and
  plots, and a results table for every card
- breadboard: C6 raised from 47 uF to 3.3 mF in the layout, wiring
  list, build steps, parts list, schematics and netlists (card 8 showed
  the half-rail reference moving with the signal)
- README: what was simulated, the numbers, and what they mean

Co-Authored-By: Claude Opus 5.5 <noreply@anthropic.com>
Claude-Session: https://claude.ai/code/session_01KoWH1xnrufgnnhp3AGqJnH
Parts:
- C6: value 47u -> 3300u
Changed lines of the file:
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@@
   (symbol (lib_id "Device:C_Polarized") (at 98 144 0) (unit 1) (in_bom yes) (on_board yes) (dnp no)
     (property "Reference" "C6" (at 100.6 143 0) (effects (font (size 1.27 1.27)) (justify left)))
-    (property "Value" "47u" (at 100.6 145.8 0) (effects (font (size 1.27 1.27)) (justify left)))
+    (property "Value" "3300u" (at 100.6 145.8 0) (effects (font (size 1.27 1.27)) (justify left)))
     (property "Footprint" "" (at 98 144 0) (effects (font (size 1.27 1.27)) hide))
     (property "Datasheet" "" (at 98 144 0) (effects (font (size 1.27 1.27)) hide))
